File: Arduino Rev 2/board/Arduino Rev 2/Arduino Rev 2.kicad_pcb (KiCad board)
At the start: 2 copper layers, 35.5 x 39.8 mm, 30 parts, among them J401 10103594-0001LF, J601 Conn_01x12_Female, J602 Conn_01x12_Female, U201 ATMEGA328-AU, U401 FT231XS-U, Y301 ECS-160-20-30B-AGL-TR

Commit message: Final Board Design
Routing:
- net +5V: track 85.0 -> 89.0 mm
- net GND: track 23.4 -> 26.6 mm, vias 13 -> 24
Other:
- board size 35.5 x 39.8 mm -> 35.5 x 40.7 mm
