File: Arduino Rev 2/board/Arduino Rev 2/CRYSTAL.sch (KiCad schematic (older format))
At the start: 3 parts, among them Y301 ECS-160-20-30B-AGL-TR

Commit message: finished Schematic
Parts:
- C301, C302: footprint Capacitor_SMD:C_0603_1608Metric_Pad1.05x0.95mm_HandSolder -> Arduino Rev 2:C_0603_1608Metric_Pad1.05x0.95mm_HandSolder
- Y301: footprint (none) -> Arduino Rev 2:ECS-160-20-30B-AGL-TR
Changed lines of the file:
@@
 $Descr A4 11693 8268
 encoding utf-8
-Sheet 3 4
+Sheet 3 6
 Title ""
 Date ""
@@
 F 0 "Y301" H 5750 4300 50  0000 L CNN
 F 1 "ECS-160-20-30B-AGL-TR" H 5550 4400 50  0000 L CNN
-F 2 "" H 5800 3500 50  0001 C CNN
+F 2 "Arduino Rev 2:ECS-160-20-30B-AGL-TR" H 5800 3500 50  0001 C CNN
 F 3 "https://ecsxtal.com/store/pdf/ecx_53b.pdf" H 5800 3500 50  0001 C CNN
 F 4 "XC2688CT-ND" H 5800 3500 50  0001 C CNN "Digikey"
@@
 $EndComp
 $Comp
-L power:GND #PWR0103
+L power:GND #PWR0302
 U 1 1 5F0CB882
 P 5800 4000
-F 0 "#PWR0103" H 5800 3750 50  0001 C CNN
+F 0 "#PWR0302" H 5800 3750 50  0001 C CNN
 F 1 "GND" H 5805 3827 50  0000 C CNN
 F 2 "" H 5800 4000 50  0001 C CNN
@@
 $EndComp
 $Comp
-L power:GND #PWR0104
+L power:GND #PWR0301
 U 1 1 5F0CC4DE
 P 5800 3000
-F 0 "#PWR0104" H 5800 2750 50  0001 C CNN
+F 0 "#PWR0301" H 5800 2750 50  0001 C CNN
 F 1 "GND" H 5805 2827 50  0000 C CNN
 F 2 "" H 5800 3000 50  0001 C CNN
@@
 F 0 "C302" H 6365 3696 50  0000 L CNN
 F 1 "22pF" H 6365 3605 50  0000 L CNN
-F 2 "Capacitor_SMD:C_0603_1608Metric_Pad1.05x0.95mm_HandSolder" H 6288 3500 50  0001 C CNN
+F 2 "Arduino Rev 2:C_0603_1608Metric_Pad1.05x0.95mm_HandSolder" H 6288 3500 50  0001 C CNN
 F 3 "~" H 6250 3650 50  0001 C CNN
 	1    6250 3650
@@
 F 0 "C301" H 5465 3696 50  0000 L CNN
 F 1 "22pF" H 5465 3605 50  0000 L CNN
-F 2 "Capacitor_SMD:C_0603_1608Metric_Pad1.05x0.95mm_HandSolder" H 5388 3500 50  0001 C CNN
+F 2 "Arduino Rev 2:C_0603_1608Metric_Pad1.05x0.95mm_HandSolder" H 5388 3500 50  0001 C CNN
 F 3 "~" H 5350 3650 50  0001 C CNN
 	1    5350 3650

Commit message: Final Board Design
Parts:
- C301, C302: Digikey (none) -> CC0603JRNPO9BN220
Changed lines of the file:
@@
 $Descr A4 11693 8268
 encoding utf-8
-Sheet 3 6
+Sheet 2 6
 Title ""
 Date ""
@@
 F 2 "Arduino Rev 2:C_0603_1608Metric_Pad1.05x0.95mm_HandSolder" H 6288 3500 50  0001 C CNN
 F 3 "~" H 6250 3650 50  0001 C CNN
+F 4 "CC0603JRNPO9BN220" H 6250 3650 50  0001 C CNN "Digikey"
 	1    6250 3650
 	1    0    0    -1
@@
 F 2 "Arduino Rev 2:C_0603_1608Metric_Pad1.05x0.95mm_HandSolder" H 5388 3500 50  0001 C CNN
 F 3 "~" H 5350 3650 50  0001 C CNN
+F 4 "CC0603JRNPO9BN220" H 5350 3650 50  0001 C CNN "Digikey"
 	1    5350 3650
 	1    0    0    -1
