File: THT Arduino/THT Arduino/THT Arduino.sch (KiCad schematic (older format))
At the start: 0 parts

Commit message: Another Commit
Changed lines of the file:
@@
 F0 "MCU" 50
 F1 "MCU.sch" 50
+F2 "XTAL1" I L 4950 1900 50
+F3 "XTAL2" I L 4950 1750 50
 $EndSheet
 $Sheet
@@
 F0 "CRYSTAL" 50
 F1 "CRYSTAL.sch" 50
+F2 "XTAL2" I R 2500 1750 50
+F3 "XTAL1" I R 2500 1900 50
+$EndSheet
+Wire Wire Line
+	2500 1900 4950 1900
+Wire Wire Line
+	2500 1750 4950 1750
+$Sheet
+S 1150 2400 1350 500
+U 5F1B5BDA
+F0 "USB to UART" 50
+F1 "USB To UART.sch" 50
 $EndSheet
 $EndSCHEMATC
