File: Nixie Clock/Nixie Clock/Microcontroller.kicad_sch (KiCad schematic)
At the start: 16 parts, among them SW1 1825910-2, U10 PIC16F15325-I/P

Commit message: Added additional parts
Parts:
- C13, C14: value (none) -> 18pF; footprint (none) -> Capacitor_THT:C_Disc_D5.0mm_W2.5mm_P2.50mm
- C15, C18: value (none) -> 0.1uF; footprint (none) -> Capacitor_THT:CP_Radial_D4.0mm_P1.50mm
- C16, C17: value (none) -> 0.01uF; footprint (none) -> Capacitor_THT:C_Disc_D5.1mm_W3.2mm_P5.00mm
- R8, R9: value (none) -> 10k; footprint (none) -> Resistor_THT:R_Axial_DIN0309_L9.0mm_D3.2mm_P12.70mm_Horizontal
- S1: value (none) -> PEC11R-4215F-S0024; footprint (none) -> digikey-footprints:Rotary_Encoder_Switched_PEC11R
- Y1: value (none) -> 12.288MHz; footprint (none) -> Crystal:Crystal_HC49-4H_Vertical
Changed lines of the file:
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@@
       (effects (font (size 1.27 1.27)) (justify left))
     )
-    (property "Value" "" (id 1) (at 118.745 69.2149 0)
-      (effects (font (size 1.27 1.27)) (justify left))
-    )
-    (property "Footprint" "" (id 2) (at 115.9002 71.755 0)
+    (property "Value" "0.1uF" (id 1) (at 118.745 69.2149 0)
+      (effects (font (size 1.27 1.27)) (justify left))
+    )
+    (property "Footprint" "Capacitor_THT:CP_Radial_D4.0mm_P1.50mm" (id 2) (at 115.9002 71.755 0)
       (effects (font (size 1.27 1.27)) hide)
     )
@@
       (effects (font (size 1.524 1.524)))
     )
-    (property "Value" "" (id 1) (at 177.8 140.97 0)
+    (property "Value" "PEC11R-4215F-S0024" (id 1) (at 177.8 140.97 0)
       (effects (font (size 1.524 1.524)))
     )
-    (property "Footprint" "" (id 2) (at 184.15 142.24 0)
+    (property "Footprint" "digikey-footprints:Rotary_Encoder_Switched_PEC11R" (id 2) (at 184.15 142.24 0)
       (effects (font (size 1.524 1.524)) (justify left) hide)
     )
@@
       (effects (font (size 1.27 1.27)) (justify left))
     )
-    (property "Value" "" (id 1) (at 68.58 62.8649 0)
-      (effects (font (size 1.27 1.27)) (justify left))
-    )
-    (property "Footprint" "" (id 2) (at 65.7352 65.405 0)
+    (property "Value" "18pF" (id 1) (at 68.58 62.8649 0)
+      (effects (font (size 1.27 1.27)) (justify left))
+    )
+    (property "Footprint" "Capacitor_THT:C_Disc_D5.0mm_W2.5mm_P2.50mm" (id 2) (at 65.7352 65.405 0)
       (effects (font (size 1.27 1.27)) hide)
     )
@@
       (effects (font (size 1.27 1.27)) (justify left))
     )
-    (property "Value" "" (id 1) (at 78.74 144.1449 0)
-      (effects (font (size 1.27 1.27)) (justify left))
-    )
-    (property "Footprint" "" (id 2) (at 77.216 143.129 90)
+    (property "Value" "10k" (id 1) (at 78.74 144.1449 0)
+      (effects (font (size 1.27 1.27)) (justify left))
+    )
+    (property "Footprint" "Resistor_THT:R_Axial_DIN0309_L9.0mm_D3.2mm_P12.70mm_Horizontal" (id 2) (at 77.216 143.129 90)
       (effects (font (size 1.27 1.27)) hide)
     )
@@
     (in_bom yes) (on_board yes) (fields_autoplaced)
     (property "Reference" "R9" (id 0) (at 140.97 135.89 90))
-    (property "Value" "" (id 1) (at 140.97 138.43 90))
-    (property "Footprint" "" (id 2) (at 141.224 141.224 90)
+    (property "Value" "10k" (id 1) (at 140.97 138.43 90))
+    (property "Footprint" "Resistor_THT:R_Axial_DIN0309_L9.0mm_D3.2mm_P12.70mm_Horizontal" (id 2) (at 141.224 141.224 90)
       (effects (font (size 1.27 1.27)) hide)
     )
@@
       (effects (font (size 1.27 1.27)) (justify left))
     )
-    (property "Value" "" (id 1) (at 196.85 137.1599 0)
-      (effects (font (size 1.27 1.27)) (justify left))
-    )
-    (property "Footprint" "" (id 2) (at 194.0052 139.7 0)
+    (property "Value" "0.1uF" (id 1) (at 196.85 137.1599 0)
+      (effects (font (size 1.27 1.27)) (justify left))
+    )
+    (property "Footprint" "Capacitor_THT:CP_Radial_D4.0mm_P1.50mm" (id 2) (at 194.0052 139.7 0)
       (effects (font (size 1.27 1.27)) hide)
     )
@@
       (effects (font (size 1.27 1.27)) (justify left))
     )
-    (property "Value" "" (id 1) (at 130.81 139.6999 0)
-      (effects (font (size 1.27 1.27)) (justify left))
-    )
-    (property "Footprint" "" (id 2) (at 127.9652 142.24 0)
+    (property "Value" "0.01uF" (id 1) (at 130.81 139.6999 0)
+      (effects (font (size 1.27 1.27)) (justify left))
+    )
+    (property "Footprint" "Capacitor_THT:C_Disc_D5.1mm_W3.2mm_P5.00mm" (id 2) (at 127.9652 142.24 0)
       (effects (font (size 1.27 1.27)) hide)
     )
@@
     (in_bom yes) (on_board yes) (fields_autoplaced)
     (property "Reference" "Y1" (id 0) (at 53.975 50.165 0))
-    (property "Value" "" (id 1) (at 53.975 52.705 0))
-    (property "Footprint" "" (id 2) (at 53.975 57.785 0)
+    (property "Value" "12.288MHz" (id 1) (at 53.975 52.705 0))
+    (property "Footprint" "Crystal:Crystal_HC49-4H_Vertical" (id 2) (at 53.975 57.785 0)
       (effects (font (size 1.27 1.27)) hide)
     )
@@
       (effects (font (size 1.27 1.27)) (justify left))
     )
-    (property "Value" "" (id 1) (at 131.445 163.8299 0)
-      (effects (font (size 1.27 1.27)) (justify left))
-    )
-    (property "Footprint" "" (id 2) (at 128.6002 166.37 0)
+    (property "Value" "0.01uF" (id 1) (at 131.445 163.8299 0)
+      (effects (font (size 1.27 1.27)) (justify left))
+    )
+    (property "Footprint" "Capacitor_THT:C_Disc_D5.1mm_W3.2mm_P5.00mm" (id 2) (at 128.6002 166.37 0)
       (effects (font (size 1.27 1.27)) hide)
     )
@@
       (effects (font (size 1.27 1.27)) (justify left))
     )
-    (property "Value" "" (id 1) (at 45.085 62.8649 0)
-      (effects (font (size 1.27 1.27)) (justify left))
-    )
-    (property "Footprint" "" (id 2) (at 42.2402 65.405 0)
-      (effects (font (size 1.27 1.27)) hide)
-    )
+    (property "Value" "18pF" (id 1) (at 45.085 62.8649 0)
+      (effects (font (size 1.27 1.27)) (justify left))
+    )
+    (property "Footprint" "Capacitor_THT:C_Disc_D5.0mm_W2.5mm_P2.50mm" (id 2) (at 42.2402 65.405 0)
+      (effects (font (size 1.27 1.27)) hide)
+    )
