File: Nixie Clock/Nixie Clock/Power Supply.kicad_sch (KiCad schematic)
At the start: 21 parts, among them J1 PJ-202A, Q1 MPSA55, U1 LM1086IT-5.0, U2 MC34063AP, U3 IRF630

Commit message: Nixie
Parts:
- C1: value 10uF -> (none); footprint Capacitor_THT:CP_Radial_D5.0mm_P2.00mm -> (none)
- C2: value 10 uF -> (none); footprint Capacitor_THT:CP_Radial_D5.0mm_P2.00mm -> (none)
- C3: value 680pF -> (none); footprint Capacitor_THT:C_Disc_D7.5mm_W4.4mm_P5.00mm -> (none)
- C4: value 220uF 25V -> (none); footprint Capacitor_THT:CP_Radial_D10.0mm_P5.00mm -> (none)
- C5: value 0.01uF -> (none); footprint Capacitor_THT:C_Disc_D12.0mm_W4.4mm_P7.75mm -> (none)
- D1: value 1N914 -> (none); footprint Diode_THT:D_DO-35_SOD27_P7.62mm_Horizontal -> (none)
- D2: value BAV21 -> (none); footprint Diode_THT:D_DO-35_SOD27_P7.62mm_Horizontal -> (none)
- L1: value 150uH 1.1A -> (none); footprint Inductor_THT:L_Radial_D12.0mm_P10.00mm_Neosid_SD12_style1 -> (none)
- Q1: value MPSA55 -> (none); footprint MPSA55:TO92127P520H787-3 -> (none)
- R1, R2: value 0.5 -> (none); footprint Resistor_THT:R_Axial_DIN0207_L6.3mm_D2.5mm_P10.16mm_Horizontal -> (none)
- R3: value 1k -> (none); footprint Resistor_THT:R_Axial_DIN0207_L6.3mm_D2.5mm_P10.16mm_Horizontal -> (none)
- R4: value 475k 1% -> (none); footprint Resistor_THT:R_Axial_DIN0207_L6.3mm_D2.5mm_P10.16mm_Horizontal -> (none)
- R5: value 13.7k 1% -> (none); footprint Resistor_THT:R_Axial_DIN0207_L6.3mm_D2.5mm_P10.16mm_Horizontal -> (none)
- R6: value 4.02k 1% -> (none); footprint Resistor_THT:R_Axial_DIN0207_L6.3mm_D2.5mm_P10.16mm_Horizontal -> (none)
- R7: value 680 1% -> (none); footprint Resistor_THT:R_Axial_DIN0207_L6.3mm_D2.5mm_P10.16mm_Horizontal -> (none)
- U3: value IRF630 -> (none); footprint IRF630:TO220V -> (none)
Changed lines of the file:
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@@
     (in_bom yes) (on_board yes) (fields_autoplaced)
     (property "Reference" "D1" (id 0) (at 161.544 63.881 0))
-    (property "Value" "1N914" (id 1) (at 161.544 66.421 0))
-    (property "Footprint" "Diode_THT:D_DO-35_SOD27_P7.62mm_Horizontal" (id 2) (at 161.544 65.786 0)
+    (property "Value" "" (id 1) (at 161.544 66.421 0))
+    (property "Footprint" "" (id 2) (at 161.544 65.786 0)
       (effects (font (size 1.27 1.27)) hide)
     )
@@
     (in_bom yes) (on_board yes) (fields_autoplaced)
     (property "Reference" "R2" (id 0) (at 125.984 41.021 90))
-    (property "Value" "0.5" (id 1) (at 125.984 43.561 90))
-    (property "Footprint" "Resistor_THT:R_Axial_DIN0207_L6.3mm_D2.5mm_P10.16mm_Horizontal" (id 2) (at 126.238 46.355 90)
+    (property "Value" "" (id 1) (at 125.984 43.561 90))
+    (property "Footprint" "" (id 2) (at 126.238 46.355 90)
       (effects (font (size 1.27 1.27)) hide)
     )
@@
       (effects (font (size 1.27 1.27)) (justify left))
     )
-    (property "Value" "150uH 1.1A" (id 1) (at 189.484 42.2909 0)
-      (effects (font (size 1.27 1.27)) (justify left))
-    )
-    (property "Footprint" "Inductor_THT:L_Radial_D12.0mm_P10.00mm_Neosid_SD12_style1" (id 2) (at 188.214 41.021 0)
+    (property "Value" "" (id 1) (at 189.484 42.2909 0)
+      (effects (font (size 1.27 1.27)) (justify left))
+    )
+    (property "Footprint" "" (id 2) (at 188.214 41.021 0)
       (effects (font (size 1.27 1.27)) hide)
     )
@@
       (effects (font (size 1.27 1.27)) (justify left))
     )
-    (property "Value" "0.5" (id 1) (at 128.651 31.4961 90)
-      (effects (font (size 1.27 1.27)) (justify left))
-    )
-    (property "Footprint" "Resistor_THT:R_Axial_DIN0207_L6.3mm_D2.5mm_P10.16mm_Horizontal" (id 2) (at 126.238 36.195 90)
+    (property "Value" "" (id 1) (at 128.651 31.4961 90)
+      (effects (font (size 1.27 1.27)) (justify left))
+    )
+    (property "Footprint" "" (id 2) (at 126.238 36.195 90)
       (effects (font (size 1.27 1.27)) hide)
     )
@@
       (effects (font (size 1.27 1.27)) (justify left))
     )
-    (property "Value" "10uF" (id 1) (at 33.02 140.0809 0)
-      (effects (font (size 1.27 1.27)) (justify left))
-    )
-    (property "Footprint" "Capacitor_THT:CP_Radial_D5.0mm_P2.00mm" (id 2) (at 30.1752 143.51 0)
+    (property "Value" "" (id 1) (at 33.02 140.0809 0)
+      (effects (font (size 1.27 1.27)) (justify left))
+    )
+    (property "Footprint" "" (id 2) (at 30.1752 143.51 0)
       (effects (font (size 1.27 1.27)) hide)
     )
@@
       (effects (font (size 1.27 1.27)) (justify left))
     )
-    (property "Value" "1k" (id 1) (at 155.702 82.9309 0)
-      (effects (font (size 1.27 1.27)) (justify left))
-    )
-    (property "Footprint" "Resistor_THT:R_Axial_DIN0207_L6.3mm_D2.5mm_P10.16mm_Horizontal" (id 2) (at 154.94 81.915 90)
+    (property "Value" "" (id 1) (at 155.702 82.9309 0)
+      (effects (font (size 1.27 1.27)) (justify left))
+    )
+    (property "Footprint" "" (id 2) (at 154.94 81.915 90)
       (effects (font (size 1.27 1.27)) hide)
     )
@@
       (effects (font (size 1.27 1.27)) (justify left))
     )
-    (property "Value" "475k 1%" (id 1) (at 210.312 63.8809 0)
-      (effects (font (size 1.27 1.27)) (justify left))
-    )
-    (property "Footprint" "Resistor_THT:R_Axial_DIN0207_L6.3mm_D2.5mm_P10.16mm_Horizontal" (id 2) (at 209.55 62.865 90)
+    (property "Value" "" (id 1) (at 210.312 63.8809 0)
+      (effects (font (size 1.27 1.27)) (justify left))
+    )
+    (property "Footprint" "" (id 2) (at 209.55 62.865 90)
       (effects (font (size 1.27 1.27)) hide)
     )
@@
       (effects (font (size 1.27 1.27)) (justify left))
     )
-    (property "Value" "0.01uF" (id 1) (at 204.216 86.7409 0)
-      (effects (font (size 1.27 1.27)) (justify left))
-    )
-    (property "Footprint" "Capacitor_THT:C_Disc_D12.0mm_W4.4mm_P7.75mm" (id 2) (at 201.8792 89.281 0)
+    (property "Value" "" (id 1) (at 204.216 86.7409 0)
+      (effects (font (size 1.27 1.27)) (justify left))
+    )
+    (property "Footprint" "" (id 2) (at 201.8792 89.281 0)
       (effects (font (size 1.27 1.27)) hide)
     )
@@
       (effects (font (size 1.27 1.27)) (justify left))
     )
-    (property "Value" "220uF 25V" (id 1) (at 168.402 43.9419 0)
-      (effects (font (size 1.27 1.27)) (justify left))
-    )
-    (property "Footprint" "Capacitor_THT:CP_Radial_D10.0mm_P5.00mm" (id 2) (at 166.3192 47.371 0)
+    (property "Value" "" (id 1) (at 168.402 43.9419 0)
+      (effects (font (size 1.27 1.27)) (justify left))
+    )
+    (property "Footprint" "" (id 2) (at 166.3192 47.371 0)
       (effects (font (size 1.27 1.27)) hide)
     )
@@
     (in_bom yes) (on_board yes) (fields_autoplaced)
     (property "Reference" "R6" (id 0) (at 232.029 73.406 90))
-    (property "Value" "4.02k 1%" (id 1) (at 232.029 75.946 90))
-    (property "Footprint" "Resistor_THT:R_Axial_DIN0207_L6.3mm_D2.5mm_P10.16mm_Horizontal" (id 2) (at 231.775 80.137 90)
+    (property "Value" "" (id 1) (at 232.029 75.946 90))
+    (property "Footprint" "" (id 2) (at 231.775 80.137 90)
       (effects (font (size 1.27 1.27)) hide)
     )
@@
       (effects (font (size 1.27 1.27)) (justify left))
     )
-    (property "Value" "IRF630" (id 1) (at 192.024 68.6241 0)
-      (effects (font (size 1.27 1.27)) (justify left))
-    )
-    (property "Footprint" "IRF630:TO220V" (id 2) (at 185.674 67.691 0)
+    (property "Value" "" (id 1) (at 192.024 68.6241 0)
+      (effects (font (size 1.27 1.27)) (justify left))
+    )
+    (property "Footprint" "" (id 2) (at 185.674 67.691 0)
       (effects (font (size 1.27 1.27)) (justify left bottom) hide)
     )
@@
     (in_bom yes) (on_board yes) (fields_autoplaced)
     (property "Reference" "D2" (id 0) (at 195.834 48.641 0))
-    (property "Value" "BAV21" (id 1) (at 195.834 51.181 0))
-    (property "Footprint" "Diode_THT:D_DO-35_SOD27_P7.62mm_Horizontal" (id 2) (at 195.834 50.546 0)
+    (property "Value" "" (id 1) (at 195.834 51.181 0))
+    (property "Footprint" "" (id 2) (at 195.834 50.546 0)
       (effects (font (size 1.27 1.27)) hide)
     )
@@
       (effects (font (size 1.27 1.27)) (justify left))
     )
-    (property "Value" "13.7k 1%" (id 1) (at 216.662 86.7409 0)
-      (effects (font (size 1.27 1.27)) (justify left))
-    )
-    (property "Footprint" "Resistor_THT:R_Axial_DIN0207_L6.3mm_D2.5mm_P10.16mm_Horizontal" (id 2) (at 215.9 85.725 90)
+    (property "Value" "" (id 1) (at 216.662 86.7409 0)
+      (effects (font (size 1.27 1.27)) (justify left))
+    )
+    (property "Footprint" "" (id 2) (at 215.9 85.725 90)
       (effects (font (size 1.27 1.27)) hide)
     )
@@
       (effects (font (size 1.27 1.27)) (justify left))
     )
-    (property "Value" "680 1%" (id 1) (at 240.792 86.1059 0)
-      (effects (font (size 1.27 1.27)) (justify left))
-    )
-    (property "Footprint" "Resistor_THT:R_Axial_DIN0207_L6.3mm_D2.5mm_P10.16mm_Horizontal" (id 2) (at 240.03 85.09 90)
+    (property "Value" "" (id 1) (at 240.792 86.1059 0)
+      (effects (font (size 1.27 1.27)) (justify left))
+    )
+    (property "Footprint" "" (id 2) (at 240.03 85.09 90)
       (effects (font (size 1.27 1.27)) hide)
     )
@@
       (effects (font (size 1.27 1.27)) (justify left))
     )
-    (property "Value" "MPSA55" (id 1) (at 171.196 76.5555 0)
-      (effects (font (size 1.27 1.27)) (justify left))
-    )
-    (property "Footprint" "MPSA55:TO92127P520H787-3" (id 2) (at 167.894 75.311 0)
+    (property "Value" "" (id 1) (at 171.196 76.5555 0)
+      (effects (font (size 1.27 1.27)) (justify left))
+    )
+    (property "Footprint" "" (id 2) (at 167.894 75.311 0)
       (effects (font (size 1.27 1.27)) (justify left bottom) hide)
     )
@@
       (effects (font (size 1.27 1.27)) (justify left))
     )
-    (property "Value" "680pF" (id 1) (at 122.936 77.8509 0)
-      (effects (font (size 1.27 1.27)) (justify left))
-    )
-    (property "Footprint" "Capacitor_THT:C_Disc_D7.5mm_W4.4mm_P5.00mm" (id 2) (at 120.5992 80.391 0)
+    (property "Value" "" (id 1) (at 122.936 77.8509 0)
+      (effects (font (size 1.27 1.27)) (justify left))
+    )
+    (property "Footprint" "" (id 2) (at 120.5992 80.391 0)
       (effects (font (size 1.27 1.27)) hide)
     )
@@
       (effects (font (size 1.27 1.27)) (justify left))
     )
-    (property "Value" "10 uF " (id 1) (at 111.76 141.3509 0)
-      (effects (font (size 1.27 1.27)) (justify left))
-    )
-    (property "Footprint" "Capacitor_THT:CP_Radial_D5.0mm_P2.00mm" (id 2) (at 108.9152 144.78 0)
-      (effects (font (size 1.27 1.27)) hide)
-    )
+    (property "Value" "" (id 1) (at 111.76 141.3509 0)
+      (effects (font (size 1.27 1.27)) (justify left))
+    )
+    (property "Footprint" "" (id 2) (at 108.9152 144.78 0)
+      (effects (font (size 1.27 1.27)) hide)
+    )

Commit message: Added additional parts
Parts:
- C1: value (none) -> 10uF; footprint (none) -> Capacitor_THT:CP_Radial_D6.3mm_P2.50mm
- C2: value (none) -> 10 uF; footprint (none) -> Capacitor_THT:CP_Radial_D6.3mm_P2.50mm
- C3: value (none) -> 680pF; footprint (none) -> Capacitor_THT:C_Disc_D3.8mm_W2.6mm_P2.50mm
- C4: value (none) -> 220uF 25V; footprint (none) -> Capacitor_THT:CP_Radial_D8.0mm_P3.50mm
- C5: value (none) -> 0.01uF; footprint (none) -> Capacitor_THT:C_Disc_D5.1mm_W3.2mm_P5.00mm
- D1: value (none) -> 1N914; footprint (none) -> Diode_THT:D_DO-35_SOD27_P7.62mm_Horizontal
- D2: value (none) -> BAV21; footprint (none) -> Diode_THT:D_DO-35_SOD27_P7.62mm_Horizontal
- L1: value (none) -> 150uH 1.1A; footprint (none) -> Inductor_THT:L_Radial_D21.0mm_P19.00mm
- R1, R2: value (none) -> 0.5; footprint (none) -> Resistor_THT:R_Axial_DIN0414_L11.9mm_D4.5mm_P15.24mm_Horizontal
- R3: value (none) -> 1k; footprint (none) -> Resistor_THT:R_Axial_DIN0207_L6.3mm_D2.5mm_P10.16mm_Horizontal
- R4: value (none) -> 475k 1%; footprint (none) -> Resistor_THT:R_Axial_DIN0204_L3.6mm_D1.6mm_P7.62mm_Horizontal
- R5: value (none) -> 13.7k 1%; footprint (none) -> Resistor_THT:R_Axial_DIN0207_L6.3mm_D2.5mm_P10.16mm_Horizontal
- R6: value (none) -> 4.02k 1%; footprint (none) -> Resistor_THT:R_Axial_DIN0204_L3.6mm_D1.6mm_P7.62mm_Horizontal
- R7: value (none) -> 680 1%; footprint (none) -> Resistor_THT:R_Axial_DIN0207_L6.3mm_D2.5mm_P10.16mm_Horizontal
- U3: value (none) -> IRF630; footprint (none) -> Package_TO_SOT_THT:TO-220-3_Vertical
Changed lines of the file:
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@@
     (in_bom yes) (on_board yes) (fields_autoplaced)
     (property "Reference" "D1" (id 0) (at 161.544 63.881 0))
-    (property "Value" "" (id 1) (at 161.544 66.421 0))
-    (property "Footprint" "" (id 2) (at 161.544 65.786 0)
+    (property "Value" "1N914" (id 1) (at 161.544 66.421 0))
+    (property "Footprint" "Diode_THT:D_DO-35_SOD27_P7.62mm_Horizontal" (id 2) (at 161.544 65.786 0)
       (effects (font (size 1.27 1.27)) hide)
     )
@@
     (in_bom yes) (on_board yes) (fields_autoplaced)
     (property "Reference" "R2" (id 0) (at 125.984 41.021 90))
-    (property "Value" "" (id 1) (at 125.984 43.561 90))
-    (property "Footprint" "" (id 2) (at 126.238 46.355 90)
+    (property "Value" "0.5" (id 1) (at 125.984 43.561 90))
+    (property "Footprint" "Resistor_THT:R_Axial_DIN0414_L11.9mm_D4.5mm_P15.24mm_Horizontal" (id 2) (at 126.238 46.355 90)
       (effects (font (size 1.27 1.27)) hide)
     )
@@
       (effects (font (size 1.27 1.27)) (justify left))
     )
-    (property "Value" "" (id 1) (at 189.484 42.2909 0)
-      (effects (font (size 1.27 1.27)) (justify left))
-    )
-    (property "Footprint" "" (id 2) (at 188.214 41.021 0)
+    (property "Value" "150uH 1.1A" (id 1) (at 189.484 42.2909 0)
+      (effects (font (size 1.27 1.27)) (justify left))
+    )
+    (property "Footprint" "Inductor_THT:L_Radial_D21.0mm_P19.00mm" (id 2) (at 188.214 41.021 0)
       (effects (font (size 1.27 1.27)) hide)
     )
@@
       (effects (font (size 1.27 1.27)) (justify left))
     )
-    (property "Value" "" (id 1) (at 128.651 31.4961 90)
-      (effects (font (size 1.27 1.27)) (justify left))
-    )
-    (property "Footprint" "" (id 2) (at 126.238 36.195 90)
+    (property "Value" "0.5" (id 1) (at 128.651 31.4961 90)
+      (effects (font (size 1.27 1.27)) (justify left))
+    )
+    (property "Footprint" "Resistor_THT:R_Axial_DIN0414_L11.9mm_D4.5mm_P15.24mm_Horizontal" (id 2) (at 126.238 36.195 90)
       (effects (font (size 1.27 1.27)) hide)
     )
@@
       (effects (font (size 1.27 1.27)) (justify left))
     )
-    (property "Value" "" (id 1) (at 33.02 140.0809 0)
-      (effects (font (size 1.27 1.27)) (justify left))
-    )
-    (property "Footprint" "" (id 2) (at 30.1752 143.51 0)
+    (property "Value" "10uF" (id 1) (at 33.02 140.0809 0)
+      (effects (font (size 1.27 1.27)) (justify left))
+    )
+    (property "Footprint" "Capacitor_THT:CP_Radial_D6.3mm_P2.50mm" (id 2) (at 30.1752 143.51 0)
       (effects (font (size 1.27 1.27)) hide)
     )
@@
       (effects (font (size 1.27 1.27)) (justify left))
     )
-    (property "Value" "" (id 1) (at 155.702 82.9309 0)
-      (effects (font (size 1.27 1.27)) (justify left))
-    )
-    (property "Footprint" "" (id 2) (at 154.94 81.915 90)
+    (property "Value" "1k" (id 1) (at 155.702 82.9309 0)
+      (effects (font (size 1.27 1.27)) (justify left))
+    )
+    (property "Footprint" "Resistor_THT:R_Axial_DIN0207_L6.3mm_D2.5mm_P10.16mm_Horizontal" (id 2) (at 154.94 81.915 90)
       (effects (font (size 1.27 1.27)) hide)
     )
@@
       (effects (font (size 1.27 1.27)) (justify left))
     )
-    (property "Value" "" (id 1) (at 210.312 63.8809 0)
-      (effects (font (size 1.27 1.27)) (justify left))
-    )
-    (property "Footprint" "" (id 2) (at 209.55 62.865 90)
+    (property "Value" "475k 1%" (id 1) (at 210.312 63.8809 0)
+      (effects (font (size 1.27 1.27)) (justify left))
+    )
+    (property "Footprint" "Resistor_THT:R_Axial_DIN0204_L3.6mm_D1.6mm_P7.62mm_Horizontal" (id 2) (at 209.55 62.865 90)
       (effects (font (size 1.27 1.27)) hide)
     )
@@
       (effects (font (size 1.27 1.27)) (justify left))
     )
-    (property "Value" "" (id 1) (at 204.216 86.7409 0)
-      (effects (font (size 1.27 1.27)) (justify left))
-    )
-    (property "Footprint" "" (id 2) (at 201.8792 89.281 0)
+    (property "Value" "0.01uF" (id 1) (at 204.216 86.7409 0)
+      (effects (font (size 1.27 1.27)) (justify left))
+    )
+    (property "Footprint" "Capacitor_THT:C_Disc_D5.1mm_W3.2mm_P5.00mm" (id 2) (at 201.8792 89.281 0)
       (effects (font (size 1.27 1.27)) hide)
     )
@@
       (effects (font (size 1.27 1.27)) (justify left))
     )
-    (property "Value" "" (id 1) (at 168.402 43.9419 0)
-      (effects (font (size 1.27 1.27)) (justify left))
-    )
-    (property "Footprint" "" (id 2) (at 166.3192 47.371 0)
+    (property "Value" "220uF 25V" (id 1) (at 168.402 43.9419 0)
+      (effects (font (size 1.27 1.27)) (justify left))
+    )
+    (property "Footprint" "Capacitor_THT:CP_Radial_D8.0mm_P3.50mm" (id 2) (at 166.3192 47.371 0)
       (effects (font (size 1.27 1.27)) hide)
     )
@@
     (in_bom yes) (on_board yes) (fields_autoplaced)
     (property "Reference" "R6" (id 0) (at 232.029 73.406 90))
-    (property "Value" "" (id 1) (at 232.029 75.946 90))
-    (property "Footprint" "" (id 2) (at 231.775 80.137 90)
+    (property "Value" "4.02k 1%" (id 1) (at 232.029 75.946 90))
+    (property "Footprint" "Resistor_THT:R_Axial_DIN0204_L3.6mm_D1.6mm_P7.62mm_Horizontal" (id 2) (at 231.775 80.137 90)
       (effects (font (size 1.27 1.27)) hide)
     )
@@
       (effects (font (size 1.27 1.27)) (justify left))
     )
-    (property "Value" "" (id 1) (at 192.024 68.6241 0)
-      (effects (font (size 1.27 1.27)) (justify left))
-    )
-    (property "Footprint" "" (id 2) (at 185.674 67.691 0)
+    (property "Value" "IRF630" (id 1) (at 192.024 68.6241 0)
+      (effects (font (size 1.27 1.27)) (justify left))
+    )
+    (property "Footprint" "Package_TO_SOT_THT:TO-220-3_Vertical" (id 2) (at 185.674 67.691 0)
       (effects (font (size 1.27 1.27)) (justify left bottom) hide)
     )
@@
     (in_bom yes) (on_board yes) (fields_autoplaced)
     (property "Reference" "D2" (id 0) (at 195.834 48.641 0))
-    (property "Value" "" (id 1) (at 195.834 51.181 0))
-    (property "Footprint" "" (id 2) (at 195.834 50.546 0)
+    (property "Value" "BAV21" (id 1) (at 195.834 51.181 0))
+    (property "Footprint" "Diode_THT:D_DO-35_SOD27_P7.62mm_Horizontal" (id 2) (at 195.834 50.546 0)
       (effects (font (size 1.27 1.27)) hide)
     )
@@
       (effects (font (size 1.27 1.27)) (justify left))
     )
-    (property "Value" "" (id 1) (at 216.662 86.7409 0)
-      (effects (font (size 1.27 1.27)) (justify left))
-    )
-    (property "Footprint" "" (id 2) (at 215.9 85.725 90)
+    (property "Value" "13.7k 1%" (id 1) (at 216.662 86.7409 0)
+      (effects (font (size 1.27 1.27)) (justify left))
+    )
+    (property "Footprint" "Resistor_THT:R_Axial_DIN0207_L6.3mm_D2.5mm_P10.16mm_Horizontal" (id 2) (at 215.9 85.725 90)
       (effects (font (size 1.27 1.27)) hide)
     )
@@
       (effects (font (size 1.27 1.27)) (justify left))
     )
-    (property "Value" "" (id 1) (at 240.792 86.1059 0)
-      (effects (font (size 1.27 1.27)) (justify left))
-    )
-    (property "Footprint" "" (id 2) (at 240.03 85.09 90)
+    (property "Value" "680 1%" (id 1) (at 240.792 86.1059 0)
+      (effects (font (size 1.27 1.27)) (justify left))
+    )
+    (property "Footprint" "Resistor_THT:R_Axial_DIN0207_L6.3mm_D2.5mm_P10.16mm_Horizontal" (id 2) (at 240.03 85.09 90)
       (effects (font (size 1.27 1.27)) hide)
     )
@@
       (effects (font (size 1.27 1.27)) (justify left))
     )
-    (property "Value" "" (id 1) (at 122.936 77.8509 0)
-      (effects (font (size 1.27 1.27)) (justify left))
-    )
-    (property "Footprint" "" (id 2) (at 120.5992 80.391 0)
+    (property "Value" "680pF" (id 1) (at 122.936 77.8509 0)
+      (effects (font (size 1.27 1.27)) (justify left))
+    )
+    (property "Footprint" "Capacitor_THT:C_Disc_D3.8mm_W2.6mm_P2.50mm" (id 2) (at 120.5992 80.391 0)
       (effects (font (size 1.27 1.27)) hide)
     )
@@
       (effects (font (size 1.27 1.27)) (justify left))
     )
-    (property "Value" "" (id 1) (at 111.76 141.3509 0)
-      (effects (font (size 1.27 1.27)) (justify left))
-    )
-    (property "Footprint" "" (id 2) (at 108.9152 144.78 0)
-      (effects (font (size 1.27 1.27)) hide)
-    )
+    (property "Value" "10 uF " (id 1) (at 111.76 141.3509 0)
+      (effects (font (size 1.27 1.27)) (justify left))
+    )
+    (property "Footprint" "Capacitor_THT:CP_Radial_D6.3mm_P2.50mm" (id 2) (at 108.9152 144.78 0)
+      (effects (font (size 1.27 1.27)) hide)
+    )
